File: minimal_ltc9111/minimal_ltc9111.kicad_pcb (KiCad board)
At the start: 4 copper layers, 65.4 x 19 mm, 36 parts, among them J1 FW-03-03-G-D-085-155, J2 FW-02-03-G-D-085-155, Q1 100 V, Q2 100 V, Q3 100 V, Q4 100.0 V, U1 LTC9111RDE-PBF

Commit message: small updates
Parts:
- added D4: 100.0 V, diode_footprints:SOD123W, F.Cu at (135.2, 112.8)
- added JP2: SolderJumper_3_Open, solder_jumper_footprints:SolderJumper-3_P1.3mm_Bridged_1_2_RoundedPad1.0x1.5mm_NumberLabels, F.Cu at (131.8, 111.5)
- moved FID2 47.0 mm to (177.8, 113.4)
- moved C5 1.52 mm to (137.9, 108.0)
- moved R3 1.14 mm to (143.0, 104.1)
- moved C1 0.51 mm to (137.9, 100.2)
Connections:
- J2 pad 2: /OUT -> /OUT_SELECTED
- J2 pad 4: /OUT -> /OUT_SELECTED
- TP3 pad 1: /OUT -> /OUT_SELECTED
Routing:
- net GND: vias 76 -> 74
- net /POWER_IN_N: vias 14 -> 13
- net /OUT_SELECTED: vias 0 -> 6
- net /OUT: vias 24 -> 14
- net /BULK_OUT: vias 17 -> 16
- added copper zone on F.Cu, net /OUT_SELECTED
- added copper zone on F.Cu, net Net-(JP2-A)

Commit message: development backup
Parts:
- removed the J1 at (183.8, 105.2)
- removed the MB1 at (179.7, 105.2)
- removed the TP2 at (179.1, 106.4)
- added J2: FW-02-03-G-D-085-155, connector_footprints:FW-02-03-G-D-085-155, F.Cu at (182.4, 100.1)
- added J3: FW-02-03-G-D-085-155, connector_footprints:FW-02-03-G-D-085-155, F.Cu at (182.4, 110.2)
- added MB2: mouse-bite-midle-50mil-200mil, mouse_bite_footprints:mouse-bite-midle-50mil-200mil, F.Cu at (179.7, 100.1)
- added MB3: mouse-bite-midle-50mil-200mil, mouse_bite_footprints:mouse-bite-midle-50mil-200mil, F.Cu at (179.7, 110.2)
- added TP3: TestPoint, test_point_footprints:TestPoint_THTPad_Castelated, F.Cu at (179.1, 99.4)
- added TP6: TestPoint, test_point_footprints:TestPoint_THTPad_Castelated, F.Cu at (179.1, 110.9)
- moved R1 8.07 mm to (143.0, 112.2), turned to 90 degrees
- moved TP5 5.71 mm to (179.1, 109.6)
- moved TP4 4.45 mm to (179.1, 100.7)
- moved C1 1.28 mm to (139.0, 99.6)
- moved C2 1.28 mm to (139.0, 107.4)
- moved D1 1.27 mm to (136.5, 112.8)
- moved FID1 1.27 mm to (132.1, 96.9)
- moved JP1 1.27 mm to (133.1, 111.5)
- moved MB1 1.27 mm to (130.2, 105.2)
- moved TP1 1.27 mm to (130.8, 104.5)
- moved TP2 1.27 mm to (130.8, 105.8)
- moved J1 1.14 mm to (127.5, 105.2)
- renumbered C5 to C2, C8 to C3, C6 to C4, C3 to C5, C9 to C6, C4 to C8, C2 to C9, D4 to D1, D1 to D2, D2 to D3, D3 to D4, FID3 to FID2, FID2 to FID3, J2 to J1, JP2 to JP1, MB2 to MB1, Q4 to Q2, Q2 to Q3, Q3 to Q4, R3 to R1, R6 to R2, R1 to R3, R2 to R4, R4 to R6, TP4 to TP1, TP3 to TP2, TP1 to TP4
Connections:
- TP5 pad 1: GND -> /POWER_IN_N
Routing:
- net GND: vias 74 -> 63
- net /POWER_IN_P: vias 13 -> 11
- net /POWER_IN_N: vias 13 -> 11
- net /OUT_SELECTED: vias 6 -> 7
- net /OUT: vias 14 -> 12
- added copper zone on In1.Cu, net /OUT_SELECTED
Other:
- board size 65.4 x 19 mm -> 60.2 x 19 mm

Commit message: development backup
Parts:
- added C10: 100 pF, capacitor_footprints:C_1812_4532Metric, F.Cu at (196.8, 102.6)
- added C11: 100 pF, capacitor_footprints:C_1812_4532Metric, F.Cu at (196.8, 107.7)
- added D5: 3.3 V, diode_footprints:SOD323, F.Cu at (191.5, 103.9)
- added D6: 58 V, diode_footprints:DO-214AA, F.Cu at (191.5, 109.5)
- added L2: 470 µH, coupled_inductor_footprints:SRF0905A, F.Cu at (181.8, 105.2)
- added R7: 10 kΩ, resistor_footprints:R_0603_1608Metric, F.Cu at (188.5, 103.1)
- added R8: 10 kΩ, resistor_footprints:R_0603_1608Metric, F.Cu at (188.5, 107.3)
- added R9: 4.7 MΩ, resistor_footprints:R_2010_5025Metric, F.Cu at (196.8, 98.0)
- added TP7: TestPoint, test_point_footprints:TestPoint_THTPad_Castelated, F.Cu at (202.7, 103.9)
- added TP8: TestPoint, test_point_footprints:TestPoint_THTPad_Castelated, F.Cu at (202.7, 105.2)
- added TP9: TestPoint, test_point_footprints:TestPoint_THTPad_Castelated, F.Cu at (202.7, 106.4)
- moved FID2 5.08 mm to (172.7, 96.9)
- moved FID3 5.08 mm to (172.7, 113.4)
- moved MB3 3.18 mm to (177.2, 112.1)
- moved MB2 3.18 mm to (177.2, 98.2)
- moved TP3 3.17 mm to (176.5, 97.5)
- moved TP4 3.17 mm to (176.5, 98.8)
- moved TP5 3.17 mm to (176.5, 111.5)
- moved TP6 3.17 mm to (176.5, 112.8)
- moved J3 2.22 mm to (181.2, 112.1), turned to 90 degrees
- moved J2 2.22 mm to (181.2, 98.2), turned to -90 degrees
Connections:
- J2 pad 1: /POWER_IN_P -> GND
- J2 pad 4: GND -> /POWER_IN_P
- J3 pad 2: /POWER_IN_N -> GND
- J3 pad 3: GND -> /POWER_IN_N
Routing:
- net Net-(D104-Pad2): track 0.00 -> 2.04 mm
- net GND: vias 63 -> 69
- net /POWER_IN_P: vias 11 -> 8
- net /POWER_IN_N: vias 11 -> 8
- added copper zone on F.Cu, net /CABLE+
- added copper zone on In1.Cu, net /CABLE+
- added copper zone on F.Cu, net /CABLE-
- added copper zone on In1.Cu, net /CABLE-
- added copper zone on F.Cu, net Earth
Other:
- board size 60.2 x 19 mm -> 77.9 x 19 mm

Commit message: development backup
Parts:
- added J4: FW-03-03-G-D-085-155, connector_footprints:FW-03-03-G-D-085-155, F.Cu at (207.4, 105.2)
- added MB6: mouse-bite-50mil-200mil, mouse_bite_footprints:mouse-bite-50mil-250mil, F.Cu at (203.4, 105.2)
- moved FID2 29.0 mm to (201.7, 96.6)
- moved FID3 29.0 mm to (201.7, 113.7)
Routing:
- net Earth: vias 0 -> 4
- net /CABLE-: vias 0 -> 3
- net /CABLE+: vias 0 -> 4
- added copper zone on B.Cu, net Earth
- added copper zone on In1.Cu, net Earth
- added copper zone on In2.Cu, net Earth
Other:
- board size 77.9 x 19 mm -> 87.1 x 19 mm
