File: minimal_ltc9111/minimal_ltc9111.kicad_sch (KiCad schematic)
At the start: 36 parts, among them J1 FW-03-03-G-D-085-155, J2 FW-02-03-G-D-085-155, Q1 100 V, Q2 100 V, Q3 100 V, Q4 100.0 V, U1 LTC9111RDE-PBF

Commit message: Switch to KiCad 9
Changed lines of the file:
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@@
 (kicad_sch
-	(version 20231120)
+	(version 20250114)
 	(generator "eeschema")
-	(generator_version "8.0")
+	(generator_version "9.0")
 	(paper "A3")
 	(junction
@@
 		)
 	)
+	(embedded_fonts no)
 )

Commit message: small updates
Parts:
- added D4: 100.0 V, diode_footprints:SOD123W, symbol UNITED_DIODES_DATA_BASE:D_PMEG10020AELR
- added JP2: SolderJumper_3_Open, solder_jumper_footprints:SolderJumper-3_P1.3mm_Bridged_1_2_RoundedPad1.0x1.5mm_NumberLabels, symbol UNITED_SOLDER_JUMPERS:SolderJumper_3_Bridged_1_2
Connections:
- net OUT: now also D4.2, JP2.3 (B); no longer J2.2, J2.4, TP3.1
- new net: D4.1, JP2.1 (A)
- new net OUT_SELECTED: J2.2, J2.4, JP2.2 (C), TP3.1
Other:
- moved on the sheet: TP3, TP4

Commit message: development backup
Parts:
- removed J1: FW-03-03-G-D-085-155, connector_footprints:FW-03-03-G-D-085-155, symbol UNITED_CONNECTORS_DATA_BASE:J_FW-03-03-G-D-085-155
- removed MB1: mouse-bite-midle-50mil-200mil, mouse_bite_footprints:mouse-bite-midle-50mil-250mil, symbol UNITED_MOUSE_BITES_DATA_BASE:mouse-bite-midle-50mil-250mil
- removed TP2: TestPoint, test_point_footprints:TestPoint_THTPad_Castelated, symbol UNITED_TEST_POINTS:TestPoint_Castelated
- added J2, J3: FW-02-03-G-D-085-155, connector_footprints:FW-02-03-G-D-085-155, symbol UNITED_CONNECTORS_DATA_BASE:J_FW-02-03-G-D-085-155
- added MB2, MB3: mouse-bite-midle-50mil-200mil, mouse_bite_footprints:mouse-bite-midle-50mil-200mil, symbol UNITED_MOUSE_BITES_DATA_BASE:mouse-bite-midle-50mil-200mil
- added TP3, TP6: TestPoint, test_point_footprints:TestPoint_THTPad_Castelated, symbol UNITED_TEST_POINTS:TestPoint_Castelated
- renumbered C5 to C2, C8 to C3, C6 to C4, C3 to C5, C9 to C6, C4 to C8, C2 to C9, D4 to D1, D1 to D2, D2 to D3, D3 to D4, FID3 to FID2, FID2 to FID3, J2 to J1, JP2 to JP1, MB2 to MB1, Q4 to Q2, Q2 to Q3, Q3 to Q4, R3 to R1, R6 to R2, R1 to R3, R2 to R4, R4 to R6, TP4 to TP1, TP3 to TP2, TP1 to TP4
Connections:
- net GND: now also J2.2, J2.4, J3.1, J3.3, TP3.1, TP6.1; no longer TP5.1
- net POWER_IN_N: now also TP5.1, J3.2, J3.4
- net POWER_IN_P: now also J2.1, J2.3
Other:
- moved on the sheet: TP4

Commit message: development backup
Parts:
- added C10, C11: 100 pF, capacitor_footprints:C_1812_4532Metric, symbol UNITED_CAPACITORS_DATA_BASE:C_C1812C101JHGACTU
- added D5: 3.3 V, diode_footprints:SOD323, symbol UNITED_DIODES_DATA_BASE:D_SP4020-01FTG-C
- added D6: 58 V, diode_footprints:DO-214AA, symbol UNITED_DIODES_DATA_BASE:D_SMBJ58CA
- added L2: 470 µH, coupled_inductor_footprints:SRF0905A, symbol UNITED_COUPLED_INDUCTORS_DATA_BASE:L_SRF0905A-471Y
- added R7, R8: 10 kΩ, resistor_footprints:R_0603_1608Metric, symbol UNITED_RESISTORS_DATA_BASE:R_ERJ-3EKF1002V
- added R9: 4.7 MΩ, resistor_footprints:R_2010_5025Metric, symbol UNITED_RESISTORS_DATA_BASE:R_CHV2010-JW-475ELF
- added TP7, TP8, TP9: TestPoint, test_point_footprints:TestPoint_THTPad_Castelated, symbol UNITED_TEST_POINTS:TestPoint_Castelated
Connections:
- net GND: now also J2.1, J3.2, R9.2; no longer J2.4, J3.3
- net POWER_IN_N: now also J3.3, L2.4, R8.2; no longer J3.2
- net POWER_IN_P: now also J2.4, L2.2, R7.2; no longer J2.1
- new net: D5.2, D6.1
- new net CABLE+: C10.1, D5.1, L2.3, R7.1, TP7.1
- new net CABLE-: C11.1, D6.2, L2.1, R8.1, TP8.1
- new net Earth: C10.2, C11.2, R9.1, TP9.1
Other:
- moved on the sheet: C1, C2, C3, C4, C5, C6, C7, C8, C9, D1, D2, D3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

Commit message: development backup
Parts:
- added J4: FW-03-03-G-D-085-155, connector_footprints:FW-03-03-G-D-085-155, symbol UNITED_CONNECTORS_DATA_BASE:J_FW-03-03-G-D-085-155
- added MB6: mouse-bite-50mil-200mil, mouse_bite_footprints:mouse-bite-50mil-250mil, symbol UNITED_MOUSE_BITES_DATA_BASE:mouse-bite-50mil-250mil
Connections:
- net CABLE+: now also J4.5, J4.6
- net CABLE-: now also J4.3, J4.4
- net Earth: now also J4.1, J4.2
Other:
- moved on the sheet: C10, C11, D5, D6, J2, J3, L2, R7, R8, R9, TP3, TP4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
